Commit message: gazebo working

File: whac_description/robots/whac.urdf.xacro (robot description, xacro)
@@ -9,16 +9,9 @@
   <xacro:include filename="$(find whac_description)/urdf/gazebo.urdf.xacro" />
   <gazebo>
-     <!--controller:gazebo_ros_controller_manager name="gazebo_ros_controller_manager" plugin="libgazebo_ros_controller_manager.so">
-          <alwaysOn>true</alwaysOn>
-          <updateRate>1000.0</updateRate>
-          <robotNamespace>dynamixel</robotNamespace>
-          <robotParam>robot_description</robotParam>
-          <interface:audio name="gazebo_ros_controller_manager_dummy_iface" />
-     </controller:gazebo_ros_controller_manager-->
-    <plugin name="gazebo_ros_control" filename="libgazebo_ros_control.so">
-      <robotNamespace>/dynamixel</robotNamespace>
-    </plugin>
+    <!--<plugin name="gazebo_ros_control" filename="libgazebo_ros_control.so">-->
+      <!--<robotNamespace>/dynamixel</robotNamespace>-->
+    <!--</plugin>-->
   </gazebo>
   <!-- Body of TurtleBot, with plates, standoffs and Create (including sim sensors) -->
-  <turtlebot_body/>
+  <whac_body/>
 </robot>

File: whac_description/urdf/body.urdf.xacro (robot description, xacro)
@@ -1,17 +1,52 @@
 <?xml version="1.0"?>
-<robot name="turtlebot_hardware" xmlns:xacro="http://ros.org/wiki/xacro">
+<robot name="whac_hardware" xmlns:xacro="http://ros.org/wiki/xacro">
     <property name="M_PI" value="3.14159"/>
     <!-- Macro for TurtleBot body. Including Gazebo extensions, but does not include Kinect -->
     <xacro:include filename="$(find whac_description)/urdf/gazebo.urdf.xacro"/>
-    <property name="base_x" value="0.33"/>
-    <property name="base_y" value="0.33"/>
-    <xacro:macro name="turtlebot_body">
+    <property name="base_x" value="0"/>
+    <property name="base_y" value="0"/>
+    <xacro:macro name="whac_body">
         <material name="GreenTB">
             <color rgba="0.0 0.8 0.0 1.0"/>
         </material>
         <!-- base_footprint is a fictitious link(frame) that is on the ground right below base_link origin, navigation stack depends on this frame -->
-        <link name="base_footprint">
+        <link name="base_link">
             <inertial>
-                <mass value="0.0001"/>
+                <mass value="10.0"/>
+                <origin xyz="0 0 0.0.025"/>
+                <inertia ixx="0.01" ixy="0.0" ixz="0.0"
+                         iyy="0.01" iyz="0.0" izz="0.5"/>
+            </inertial>
+            <visual>
+                <origin xyz=" 0 0 0.025" rpy="0 0 0"/>
+                <geometry>
+                    <cylinder length="0.05" radius="0.15"/>
+                </geometry>
+            </visual>
+            <collision>
+                <origin xyz="0.0 0.0 0.025" rpy="0 0 0"/>
+                <geometry>
+                    <cylinder length="0.05" radius="0.15"/>
+                </geometry>
+            </collision>
+        </link>
+        <joint name="laser_joint" type="fixed">
+            <!-- correct values for rpy are ${M_PI} 0 0 (real laser is upside down), but then gmapping doesn't work -->
+            <origin xyz="0.085 0 0.1" rpy="0 0 -${M_PI}/2.0"/>
+            <parent link="base_link"/>
+            <child link="laser"/>
+        </joint>
+        <link name="laser">
+            <visual>
+                <origin xyz="0 0 0" rpy="0 0 0"/>
+                <geometry>
+                    <cylinder radius="0.035" length="0.023"/>
+                </geometry>
+                <material name="blue">
+                    <color rgba="0 0 .8 1"/>
+                </material>
+            </visual>
+            <inertial>
+                <mass value="0.5"/>
                 <origin xyz="0 0 0"/>
                 <inertia ixx="0.0001" ixy="0.0" ixz="0.0"
@@ -19,72 +54,10 @@
                          izz="0.0001"/>
             </inertial>
-            <visual>
+            <collision>
                 <origin xyz="0 0 0" rpy="0 0 0"/>
                 <geometry>
-                    <box size="0.001 0.001 0.001"/>
-                </geometry>
-                <material name="GreenTB"/>
-            </visual>
-            <collision>
-                <origin xyz="0 0 0.017" rpy="0 0 0"/>
-                <geometry>
-                    <box size="0.001 0.001 0.001"/>
+                    <cylinder radius="0.035" length="0.023"/>
                 </geometry>
             </collision>
-        </link>
-        <link name="base_link">
-            <inertial>
-                <mass value="10.0"/>
-                <origin xyz="0 0 0.0"/>
-                <inertia ixx="0.01" ixy="0.0" ixz="0.0"
-                         iyy="0.01" iyz="0.0" izz="0.5"/>
-            </inertial>
-            <visual>
-                <origin xyz=" 0 0 0.0308" rpy="0 0 0"/>
-                <geometry>
-                    <cylinder length="0.0611632" radius="0.016495"/>
-                </geometry>
-            </visual>
-            <collision>
-                <origin xyz="0.0 0.0 0.0308" rpy="0 0 0"/>
-                <geometry>
-                    <cylinder length="0.0611632" radius="0.016495"/>
-                </geometry>
-            </collision>
-        </link>
-        <joint name="base_footprint_joint" type="fixed">
-            <origin xyz="0 0 0.017" rpy="0 0 0"/>
-            <parent link="base_footprint"/>
-            <child link="base_link"/>
-        </joint>
-        <joint name="laser_joint" type="fixed">
-            <!-- correct values for rpy are ${M_PI} 0 0 (real laser is upside down), but then gmapping doesn't work -->
-            <origin xyz="0.26 0 0.025" rpy="0 0 0"/>
-            <parent link="base_link"/>
-            <child link="laser"/>
-        </joint>
-        <link name="laser">
-            <visual>
-                <origin xyz="0 0 0.05" rpy="0 0 0"/>
-                <geometry>
-                    <box size="0.1 0.1 0.15"/>
-                </geometry>
-                <material name="blue">
-                    <color rgba="0 0 .8 1"/>
-                </material>
-            </visual>
-            <collision>
-                <origin xyz="0 0 0.05" rpy="0 0 0"/>
-                <geometry>
-                    <box size="0.1 0.1 0.15"/>
-                </geometry>
-            </collision>
-            <inertial>
-                <mass value="0.5"/>
-                <origin xyz="0 0 0.05"/>
-                <inertia ixx="0.0001" ixy="0.0" ixz="0.0"
-                         iyy="0.0001" iyz="0.0"
-                         izz="0.0001"/>
-            </inertial>
         </link>
         <gazebo reference="laser">
@@ -116,5 +89,5 @@
         </link>
         <joint name="front_left_wheel_joint" type="continuous">
-            <origin xyz="0.1 0.13 0.015" rpy="0 0 0"/>
+            <origin xyz="0.1 0.13 0" rpy="0 0 0"/>
             <parent link="base_link"/>
             <child link="front_left_wheel_link"/>
@@ -145,5 +118,5 @@
         </link>
         <joint name="front_right_wheel_joint" type="continuous">
-            <origin xyz="0.1 -0.13 0.015" rpy="0 0 0"/>
+            <origin xyz="0.1 -0.13 0" rpy="0 0 0"/>
             <parent link="base_link"/>
             <child link="front_right_wheel_link"/>
@@ -174,5 +147,5 @@
         </link>
         <joint name="back_left_wheel_joint" type="continuous">
-            <origin xyz="-0.1 0.13 0.015" rpy="0 0 0"/>
+            <origin xyz="-0.1 0.13 0" rpy="0 0 0"/>
             <parent link="base_link"/>
             <child link="back_left_wheel_link"/>
@@ -203,5 +176,5 @@
         </link>
         <joint name="back_right_wheel_joint" type="continuous">
-            <origin xyz="-0.1 -0.13 0.015" rpy="0 0 0"/>
+            <origin xyz="-0.1 -0.13 0" rpy="0 0 0"/>
             <parent link="base_link"/>
             <child link="back_right_wheel_link"/>

File: whac_description/urdf/gazebo.urdf.xacro (robot description, xacro)
@@ -6,5 +6,5 @@
     <xacro:macro name="whac_sim_laser">
         <gazebo reference="laser">
-            <sensor type="gpu_ray" name="head_rplidar_sensor">
+            <sensor type="ray" name="head_rplidar_sensor">
                 <pose>0 0 0 0 0 0</pose>
                 <visualize>false</visualize>
@@ -13,5 +13,5 @@
                     <scan>
                         <horizontal>
-                            <samples>720</samples>
+                            <samples>360</samples>
                             <resolution>1</resolution>
                             <min_angle>-3.14159265</min_angle>
@@ -19,4 +19,5 @@
                         </horizontal>
                     </scan>
+                    <updateRate>10.0</updateRate>
                     <range>
                         <min>0.2</min>
@@ -30,5 +31,5 @@
                     </noise>
                 </ray>
-                <plugin name="gazebo_ros_head_rplidar_controller" filename="libgazebo_ros_gpu_laser.so">
+                <plugin name="gazebo_ros_head_rplidar_controller" filename="libgazebo_ros_laser.so">
                     <topicName>scan</topicName>
                     <frameName>laser</frameName>
@@ -39,20 +40,18 @@
     <xacro:macro name="whac_sim_create">
         <gazebo>
-            <gazebo>
-                <plugin name="skid_steer_drive_controller" filename="libgazebo_ros_skid_steer_drive.so">
-                    <updateRate>100.0</updateRate>
-                    <robotNamespace>/</robotNamespace>
-                    <leftFrontJoint>front_left_wheel_joint</leftFrontJoint>
-                    <rightFrontJoint>front_right_wheel_joint</rightFrontJoint>
-                    <leftRearJoint>back_left_wheel_joint</leftRearJoint>
-                    <rightRearJoint>back_right_wheel_joint</rightRearJoint>
-                    <wheelSeparation>0.44</wheelSeparation>
-                    <wheelDiameter>0.215</wheelDiameter>
-                    <robotBaseFrame>base_link</robotBaseFrame>
-                    <torque>20</torque>
-                    <topicName>cmd_vel</topicName>
-                    <broadcastTF>false</broadcastTF>
-                </plugin>
-            </gazebo>
+            <plugin name="skid_steer_drive_controller" filename="libgazebo_ros_skid_steer_drive.so">
+                <updateRate>100.0</updateRate>
+                <robotNamespace>/</robotNamespace>
+                <leftFrontJoint>front_left_wheel_joint</leftFrontJoint>
+                <rightFrontJoint>front_right_wheel_joint</rightFrontJoint>
+                <leftRearJoint>back_left_wheel_joint</leftRearJoint>
+                <rightRearJoint>back_right_wheel_joint</rightRearJoint>
+                <wheelSeparation>0.44</wheelSeparation>
+                <wheelDiameter>0.215</wheelDiameter>
+                <robotBaseFrame>base_link</robotBaseFrame>
+                <torque>20</torque>
+                <topicName>/cmd_vel</topicName>
+                <broadcastTF>false</broadcastTF>
+            </plugin>
         </gazebo>
     </xacro:macro>
